File: ac-adapter.sch (EAGLE design)
At the start: 67 parts, among them IC1 BM1Q011, IC2 TL431, Q1 TLP621-1, Q2 600V5A, T1 COMMON_FILTER-SU10VFC, T2 TRANSFORMAER_FLYBACK-PQ2620-2

Commit message: PFCコントローラーを使う
Parts:
- added C21: 1000p, my_rcl:C-1608
- added D3: 1N4148, my_rcl:DIODE-1N4148W
- added R19, R22: DNP, my_rcl:R-1608
- added R20: 100k, my_rcl:R-1608
- added R21, R23: 240k, my_rcl:R-1608
- IC1: value BM1Q011 -> NCP1608; device my_ic:BM1Q011 -> my_ic:NCP1608
- R15: value 10k -> DNP; device my_rcl:R-2012 -> my_rcl:R-1608
- R4: value 10k -> 47k
- R5: value 1.5k -> DNP
- SJ1, SJ2: device Connector_Robotech:SJ1608 -> my_rcl:SJ-1608
Connections:
- new net N$24: D3.A, IC1.FB, R20.1
- new net N$30: R15.2, R22.1
- new net N$31: R21.2, R23.1
- net N$13: now also IC1.DRV; no longer IC1.OUT
- net N$19: now also IC1.COMP; no longer IC1.FB
- net N$5: now also C21.1, IC1.CT, R19.2; no longer IC1.VH
- net N$7: now also IC1.ZCD; no longer IC1.ZT
- net PGND: now also C21.2, D3.K, R19.1
- net VCC: now also R20.2, R21.1
- net VP: now also R22.2, R23.2; no longer R15.2
Other:
- moved on the sheet: C1, C18, C19, C2, C3, C4, C6, C7, D1, F1, FB1, HT1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
